File: Hardware/EmbedLinux/EmbedLinux.kicad_sch (KiCad schematic)
At the start: 0 parts

Commit message: small updates to layout and idea
Other:
- added sheet ETH (eth.kicad_sch)
- added sheet GPIOs (gpios.kicad_sch)
- added sheet MPU (MPU.kicad_sch)
- added sheet Memory (memory.kicad_sch)
- added sheet PMIC (pmic.kicad_sch)
Changed lines of the file:
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@@
 (kicad_sch (version 20211123) (generator eeschema)
   (paper "A4")
+  (sheet (at 120.65 91.44) (size 24.13 21.59) (fields_autoplaced)
+    (stroke (width 0.1524) (type solid) (color 0 0 0 0))
+    (fill (color 0 0 0 0.0000))
+    (property "Sheet name" "MPU" (id 0) (at 120.65 90.7284 0)
+      (effects (font (size 1.27 1.27)) (justify left bottom))
+    )
+    (property "Sheet file" "MPU.kicad_sch" (id 1) (at 120.65 113.6146 0)
+      (effects (font (size 1.27 1.27)) (justify left top))
+    )
+  )
+  (sheet (at 52.07 43.18) (size 40.64 33.02) (fields_autoplaced)
+    (stroke (width 0.1524) (type solid) (color 0 0 0 0))
+    (fill (color 0 0 0 0.0000))
+    (property "Sheet name" "ETH" (id 0) (at 52.07 42.4684 0)
+      (effects (font (size 1.27 1.27)) (justify left bottom))
+    )
+    (property "Sheet file" "eth.kicad_sch" (id 1) (at 52.07 76.7846 0)
+      (effects (font (size 1.27 1.27)) (justify left top))
+    )
+  )
+  (sheet (at 132.08 135.89) (size 31.75 17.78) (fields_autoplaced)
+    (stroke (width 0.1524) (type solid) (color 0 0 0 0))
+    (fill (color 0 0 0 0.0000))
+    (property "Sheet name" "Memory" (id 0) (at 132.08 135.1784 0)
+      (effects (font (size 1.27 1.27)) (justify left bottom))
+    )
+    (property "Sheet file" "memory.kicad_sch" (id 1) (at 132.08 154.2546 0)
+      (effects (font (size 1.27 1.27)) (justify left top))
+    )
+  )
+  (sheet (at 71.12 100.33) (size 31.75 25.4) (fields_autoplaced)
+    (stroke (width 0.1524) (type solid) (color 0 0 0 0))
+    (fill (color 0 0 0 0.0000))
+    (property "Sheet name" "PMIC" (id 0) (at 71.12 99.6184 0)
+      (effects (font (size 1.27 1.27)) (justify left bottom))
+    )
+    (property "Sheet file" "pmic.kicad_sch" (id 1) (at 71.12 126.3146 0)
+      (effects (font (size 1.27 1.27)) (justify left top))
+    )
+  )
+  (sheet (at 170.18 41.91) (size 59.69 36.83) (fields_autoplaced)
+    (stroke (width 0.1524) (type solid) (color 0 0 0 0))
+    (fill (color 0 0 0 0.0000))
+    (property "Sheet name" "GPIOs" (id 0) (at 170.18 41.1984 0)
+      (effects (font (size 1.27 1.27)) (justify left bottom))
+    )
+    (property "Sheet file" "gpios.kicad_sch" (id 1) (at 170.18 79.3246 0)
+      (effects (font (size 1.27 1.27)) (justify left top))
+    )
+  )
   (sheet_instances
     (path "/" (page "1"))
+    (path "/4703a239-d4dc-44af-bbd0-3f8d3fbe6158" (page "2"))
+    (path "/d3386e79-5912-4c1e-af9b-28b2142f98fa" (page "3"))
+    (path "/7e98c23d-dc0e-4a73-92e6-2c87e92dac68" (page "4"))
+    (path "/91ec1303-b32e-4ed5-b959-68fb96488392" (page "5"))
+    (path "/87342b29-5d5c-4c82-a596-e5bb9271758b" (page "6"))
   )
 )
